File: Eagle/CMM.PCB.v1.0.sch (EAGLE design)
At the start: 2 parts

Commit message: Update Corrected Schematic and Board files
Parts:
- removed LED1: RGBLED_CA-5MM, adafruit:RGBLED_CA-5MM
- removed MKRCAN: -, MKRcan:ARDUINO-UTILITY_MKRBOARD
- added JP1: (no value), microbuilder:HEADER-1X16ROUND
- added JP2: (no value), microbuilder:HEADER-1X870MIL
- added JP3: (no value), microbuilder:HEADER-1X12
- added LED2: RGBLED_CA-5MM, adafruit:RGBLED_CA-5MM
- added MKR1: -, adafruit:ARDUINO-UTILITY_MKRBOARDOUTLINE
- added SW1: SPST_TACT-KMR2, adafruit:SPST_TACT-KMR2
Connections:
- new net GND: JP1.12, JP2.7, LED2.VCC, MKR1.GND, SW1.S, SW1.S1
- new net RST: JP1.16, SW1.P, SW1.P1
- net N$1: now also JP3.9, MKR1.3; no longer MKRCAN.3
- net N$10: now also JP3.7, LED2.GREEN; no longer LED1.GREEN
- net N$11: now also JP3.8, LED2.BLUE; no longer LED1.BLUE
- net N$2: now also JP2.4, JP3.12, MKR1.7; no longer MKRCAN.7
- net N$3: now also JP1.5, MKR1.8/MOSI; no longer MKRCAN.8/MOSI
- net N$4: now also JP1.6, MKR1.9/SCK; no longer MKRCAN.9/SCK
- net N$5: now also JP1.4, MKR1.10/MISO; no longer MKRCAN.10/MISO
- net N$6: now also JP1.15, JP2.8, MKR1.VCC; no longer MKRCAN.VCC
- net N$7: now also JP3.3, MKR1.5V, MKR1.VIN; no longer MKRCAN.5V, MKRCAN.VIN
- net N$8: now also JP3.6, LED2.RED; no longer LED1.VCC, MKRCAN.GND
- net N$9: now also JP2.5, JP3.11; no longer LED1.RED
Other:
- note removed: "1"
- note removed: "10"
- note removed: "11"
- note removed: "12"
- note removed: "13"
- note removed: "14"
- note removed: "15"
- note removed: "16"
- note removed: "2"
- note removed: "3"
- note removed: "3V"
- note removed: "4"
- note removed: "5"
- note removed: "6"
- note removed: "7"
- note removed: "8"
- note removed: "9"
- note removed: "A0"
- note removed: "A1"
- note removed: "A2"
- note removed: "A3"
- note removed: "A4"
- note removed: "A5"
- note removed: "ADAFRUIT FEATHER 32U4"
- note removed: "ARf"
- note removed: "EN"
- note removed: "EXT ANT"
- note removed: "FRAM"
- note removed: "GND"
- note removed: "IO1"
- note removed: "IO2"
- note removed: "IO3"
- note removed: "MISO"
- note removed: "MOSI"
- note removed: "OBD-II"
- note removed: "RST"
- note removed: "RX"
- note removed: "SCK"
- note removed: "SCL"
- note removed: "SDA"
- note removed: "TX"
- note removed: "USB"
- note removed: "VBAT"
- note removed: "VCC"
- note removed: "WP"
