File: Eagle Files/CMM.PCB.v1.0.brd (EAGLE design)
At the start: 70.8 x 54 mm, 6 parts, among them SW1 SPST_TACT-KMR2

Commit message: Board and Schematic files
Connections:
- removed net RST: JP1.16, SW1.1, SW1.3
- new net SIGNAL: JP1.12, SW1.1, SW1.3
- net GND: now also JP1.13; no longer JP1.12
Routing:
- net SIGNAL: track 0.00 -> 26.4 mm
- net RST: track 20.6 -> 0.00 mm
- net N$10: track 64.8 -> 57.5 mm
- net N$8: track 54.4 -> 61.0 mm
- net GND: track 125.3 -> 120.2 mm
- net N$11: track 64.4 -> 62.0 mm
